File: esp32s2-co2-monitor/kicad-src/esp32s2-co2-monitor.kicad_sch (KiCad schematic)
At the start: 94 parts, among them J1 USB_C, J2 Conn_01x10_MountingPin, J3 Conn_01x07_Male, J4 JST, SW1 SW_Push, SW2 SW_Push, SW3 SW_Push, U1 USBLC6-2, U2 TLV62569DRL, U3 ESP32-S2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

Commit message: Update esp32s2 co2 monitor
Parts:
- added C23: 2.2uF, Capacitor_SMD:C_0402_1005Metric, symbol Device:C
- added C24: 22uF, Capacitor_SMD:C_0603_1608Metric, symbol Device:C
- added C25: 4.7uF, Capacitor_SMD:C_0402_1005Metric, symbol Device:C
- added L3: 2.2uH, Inductor_SMD:L_0805_2012Metric, symbol Device:L_Small
- added R18: 36.5k, Resistor_SMD:R_0402_1005Metric, symbol Device:R
- added R19: 16.2k, Resistor_SMD:R_0402_1005Metric, symbol Device:R
- added U7: TPS63900, Package_SON:WSON-10-1EP_2.5x2.5mm_P0.5mm_EP1.2x2mm_ThermalVias, symbol gsd-kicad:TPS63900
Connections:
- net +3V3: no longer C18.1, J2.6 (Pin_6), J2.7 (Pin_7)
- net GND: now also C23.2, C24.2, C25.2, R18.1, R19.1, U7.11 (PGND), U7.5 (CFG3), U7.8 (GND)
- net V_SYS: now also C25.1, U7.1 (EN), U7.10 (VIN), U7.2 (SEL)
- new net: R18.2, U7.3 (CFG1)
- new net: R19.2, U7.4 (CFG2)
- new net: L3.1, U7.9 (L1)
- new net: L3.2, U7.7 (L2)
- new net +5V: C18.1, C23.1, C24.1, J2.6 (Pin_6), J2.7 (Pin_7), U7.6 (VOUT)
Other:
- moved on the sheet: C2, C3, C4, R10, R4, R5, R8, R9, SW1, SW2, SW3, U1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
