File: syzygy-sgmii/kicad-src/pMCU.kicad_sch (KiCad schematic)
At the start: 5 parts, among them J3 TagConnect, U2 ATtiny44A-MMH

Commit message: Finish syzygy-sgmii
Other:
- title: SYZYGY PCIe x4 -> SYZYGY SGMII
Changed lines of the file:
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@@
   (paper "A4")
   (title_block
-    (title "SYZYGY PCIe x4")
-    (date "2020-12-04")
+    (title "SYZYGY SGMII")
+    (date "2020-12-08")
     (rev "r1.0")
     (company "GsD - @gregdavill")

Commit message: syzygy-sgmii: Add BOM values to project
Parts:
- C10: Mfg Samsung Electro-Mechanics -> Yageo; PN CL05A105KP5NNNC -> CC0402KRX5R8BB105
- C9: Mfg Samsung Electro-Mechanics -> Yageo; PN CL05B104KP5NNNC -> CC0402JRX7R7BB104
- R15: Mfg Stackpole Electronics Inc -> Yageo; PN RMCF0402FT10K0 -> AC0402FR-0710KL
Changed lines of the file:
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@@
-(kicad_sch (version 20201015) (generator eeschema)
+(kicad_sch (version 20210126) (generator eeschema)
   (paper "A4")
   (title_block
@@
       (effects (font (size 1.27 1.27)) hide)
     )
+    (pin "1")
   )
   (symbol (lib_id "gkl_power:GND") (at 194.31 100.33 0) (mirror y) (unit 1)
@@
       (effects (font (size 1.27 1.27)) hide)
     )
+    (pin "1")
   )
   (symbol (lib_id "gkl_power:GND") (at 207.01 100.33 0) (mirror y) (unit 1)
@@
       (effects (font (size 1.27 1.27)) hide)
     )
+    (pin "1")
   )
   (symbol (lib_id "gkl_power:GND") (at 213.36 128.27 0) (mirror y) (unit 1)
@@
       (effects (font (size 1.27 1.27)) hide)
     )
+    (pin "1")
   )
   (symbol (lib_id "gkl_power:+3V3") (at 132.08 68.58 0) (mirror y) (unit 1)
@@
       (effects (font (size 1.27 1.27)) hide)
     )
+    (pin "1")
   )
   (symbol (lib_id "gkl_power:+3V3") (at 156.21 68.58 0) (mirror y) (unit 1)
@@
       (effects (font (size 1.27 1.27)) hide)
     )
+    (pin "1")
   )
   (symbol (lib_id "gkl_power:+3V3") (at 194.31 85.09 0) (mirror y) (unit 1)
@@
       (effects (font (size 1.27 1.27)) hide)
     )
+    (pin "1")
   )
   (symbol (lib_id "gkl_power:+3V3") (at 207.01 85.09 0) (mirror y) (unit 1)
@@
       (effects (font (size 1.27 1.27)) hide)
     )
+    (pin "1")
   )
   (symbol (lib_id "gkl_power:+3V3") (at 213.36 116.84 0) (mirror y) (unit 1)
@@
       (effects (font (size 1.27 1.27)) hide)
     )
+    (pin "1")
   )
   (symbol (lib_id "Device:R") (at 132.08 74.93 0) (unit 1)
@@
       (effects (font (size 1.27 1.27)) hide)
     )
-    (property "Mfg" "Stackpole Electronics Inc" (id 4) (at 0 149.86 0)
-      (effects (font (size 1.27 1.27)) hide)
-    )
-    (property "PN" "RMCF0402FT10K0" (id 5) (at 0 149.86 0)
-      (effects (font (size 1.27 1.27)) hide)
-    )
+    (property "Mfg" "Yageo" (id 4) (at 0 149.86 0)
+      (effects (font (size 1.27 1.27)) hide)
+    )
+    (property "PN" "AC0402FR-0710KL" (id 5) (at 0 149.86 0)
+      (effects (font (size 1.27 1.27)) hide)
+    )
+    (pin "1")
+    (pin "2")
   )
   (symbol (lib_id "Device:C") (at 194.31 92.71 0) (unit 1)
@@
       (effects (font (size 1.27 1.27)) hide)
     )
-    (property "PN" "CL05B104KP5NNNC" (id 4) (at -1.27 185.42 0)
-      (effects (font (size 1.27 1.27)) hide)
-    )
-    (property "Mfg" "Samsung Electro-Mechanics" (id 5) (at -1.27 185.42 0)
-      (effects (font (size 1.27 1.27)) hide)
-    )
+    (property "PN" "CC0402JRX7R7BB104" (id 4) (at -1.27 185.42 0)
+      (effects (font (size 1.27 1.27)) hide)
+    )
+    (property "Mfg" "Yageo" (id 5) (at -1.27 185.42 0)
+      (effects (font (size 1.27 1.27)) hide)
+    )
+    (pin "1")
+    (pin "2")
   )
   (symbol (lib_id "Device:C") (at 207.01 92.71 0) (unit 1)
@@
       (effects (font (size 1.27 1.27)) hide)
     )
-    (property "PN" "CL05A105KP5NNNC" (id 4) (at 0 185.42 0)
-      (effects (font (size 1.27 1.27)) hide)
-    )
-    (property "Mfg" "Samsung Electro-Mechanics" (id 5) (at 0 185.42 0)
-      (effects (font (size 1.27 1.27)) hide)
-    )
+    (property "PN" "CC0402KRX5R8BB105" (id 4) (at 0 185.42 0)
+      (effects (font (size 1.27 1.27)) hide)
+    )
+    (property "Mfg" "Yageo" (id 5) (at 0 185.42 0)
+      (effects (font (size 1.27 1.27)) hide)
+    )
+    (pin "1")
+    (pin "2")
   )
   (symbol (lib_id "Connector_Generic:Conn_02x03_Odd_Even") (at 201.93 123.19 0) (unit 1)
@@
       (effects (font (size 1.27 1.27)) hide)
     )
+    (pin "1")
+    (pin "2")
+    (pin "3")
+    (pin "4")
+    (pin "5")
+    (pin "6")
   )
   (symbol (lib_id "SyzygyLVDSPod-rescue:ATtiny44A-MMH-MCU_Microchip_ATtiny") (at 156.21 97.79 0) (mirror y) (unit 1)
@@
       (effects (font (size 1.27 1.27)) hide)
     )
+    (pin "1")
+    (pin "10")
+    (pin "11")
+    (pin "12")
+    (pin "13")
+    (pin "14")
+    (pin "15")
+    (pin "16")
+    (pin "17")
+    (pin "18")
+    (pin "19")
+    (pin "2")
+    (pin "20")
+    (pin "21")
+    (pin "3")
+    (pin "4")
+    (pin "5")
+    (pin "6")
+    (pin "7")
+    (pin "8")
+    (pin "9")
   )
 )
