File: syzygy-sgmii/kicad-src/syzygy-sgmii.kicad_pcb (KiCad board)
At the start: 4 copper layers, 50 x 70 mm, 97 parts, among them CON1 JD1_0001NL, J1 SYZYGY-TXR-4, J3 TagConnect, U1 DP83867C, U2 ATtiny44A-MMH, U3 TLV62569DRL, U4 TLV62569DRL, U5 TLV62569DRL, Y1 25MHz

Commit message: Finish syzygy-sgmii
Parts:
- removed the R1 at (127.5, 91.2)
- added C32: 0.1uF, Capacitor_SMD:C_0402_1005Metric, F.Cu at (134.9, 84.8)
- added R16: 100R, Resistor_SMD:R_0402_1005Metric, F.Cu at (131.8, 87.1)
- added R17: 10k, Resistor_SMD:R_0402_1005Metric, F.Cu at (119.3, 129.7)
- added R18: 2.49k, Resistor_SMD:R_0402_1005Metric, F.Cu at (119.3, 130.7)
- added U6: TPD4EUSB30, Package_SON:USON-10_2.5x1.0mm_P0.5mm, F.Cu at (128.2, 127.4)
- added U7: TPD4EUSB30, Package_SON:USON-10_2.5x1.0mm_P0.5mm, F.Cu at (131.2, 127.4)
- added X1: SG3225VAN, Oscillator:Oscillator_SMD_Silicon_Labs_LGA-6_2.5x3.2mm_P1.25mm, F.Cu at (132.4, 84.9)
- moved C3 1.75 mm to (133.2, 129.7)
- moved C4 1.75 mm to (138.8, 129.7)
- moved Y1 1.75 mm to (136.0, 128.9)
Connections:
- net /SGMII_SIN_N renamed /SGMII_SI_N
- net /SGMII_SIN_P renamed /SGMII_SI_P
- net /SGMII_SON_N renamed /SGMII_SO_N
- net /SGMII_SON_P renamed /SGMII_SO_P
- net /_SGMII_SIN_N renamed /_SGMII_SI_N
- net /_SGMII_SIN_P renamed /_SGMII_SI_P
- net /_SGMII_SON_N renamed /_SGMII_SO_N
- net /_SGMII_SON_P renamed /_SGMII_SO_P
- CON1 pad 11: no_connect_92 -> no_connect_91
- U1 pad 25: no_connect_93 -> GND
- U1 pad 26: no_connect_94 -> GND
- U1 pad 29: no_connect_95 -> GND
- U1 pad 32: no_connect_96 -> no_connect_92
- U1 pad 33: no_connect_97 -> no_connect_93
- U1 pad 34: no_connect_98 -> no_connect_94
- U1 pad 37: no_connect_99 -> GND
- U1 pad 38: no_connect_100 -> no_connect_95
- U2 pad 10: no_connect_101 -> no_connect_96
- U2 pad 17: no_connect_102 -> no_connect_97
- U2 pad 18: no_connect_103 -> no_connect_98
- U2 pad 19: no_connect_104 -> no_connect_99
- U2 pad 6: no_connect_105 -> no_connect_100
- U2 pad 7: no_connect_106 -> no_connect_101
- U3 pad 6: no_connect_107 -> no_connect_102
- U4 pad 6: no_connect_108 -> no_connect_103
- U5 pad 6: no_connect_109 -> no_connect_104
Routing:
- net /VCCIO: track 94.6 -> 127.9 mm
- net /REFCLK_P: track 18.0 -> 9.43 mm
- net /REFCLK_N: track 17.5 -> 9.45 mm
- net GND: track 53.1 -> 57.9 mm, vias 48 -> 60
- net +3V3: track 42.0 -> 46.7 mm, vias 5 -> 6
- net /LED0: track 29.3 -> 32.9 mm
- net Net-(C4-Pad1): track 11.7 -> 13.4 mm
- net Net-(C3-Pad1): track 12.6 -> 14.4 mm

Commit message: syzygy-sgmii: Add BOM values to project
Parts:
- R2: value 84k5 -> 10K
- R3, R5: value 100k -> 15K
- R4: value 84k5 -> 47.5K
- R6: value 84k5 -> 20K
- R7: value 100k -> 10K
Connections:
- CON1 pad 11: no_connect_91 -> unconnected-(CON1-Pad11)
- J1 pad 10: Net-(J1-Pad10) -> unconnected-(J1-Pad10)
- J1 pad 11: Net-(J1-Pad11) -> unconnected-(J1-Pad11)
- J1 pad 12: Net-(J1-Pad12) -> unconnected-(J1-Pad12)
- J1 pad 25: Net-(J1-Pad25) -> unconnected-(J1-Pad25)
- J1 pad 26: Net-(J1-Pad26) -> unconnected-(J1-Pad26)
- J1 pad 27: Net-(J1-Pad27) -> unconnected-(J1-Pad27)
- J1 pad 28: Net-(J1-Pad28) -> unconnected-(J1-Pad28)
- J1 pad 29: Net-(J1-Pad29) -> unconnected-(J1-Pad29)
- J1 pad 30: Net-(J1-Pad30) -> unconnected-(J1-Pad30)
- J1 pad 31: Net-(J1-Pad31) -> unconnected-(J1-Pad31)
- J1 pad 32: Net-(J1-Pad32) -> unconnected-(J1-Pad32)
- J1 pad 37: Net-(J1-Pad37) -> unconnected-(J1-Pad37)
- J1 pad 38: Net-(J1-Pad38) -> unconnected-(J1-Pad38)
- J1 pad 9: Net-(J1-Pad9) -> unconnected-(J1-Pad9)
- U1 pad 32: no_connect_92 -> unconnected-(U1-Pad32)
- U1 pad 33: no_connect_93 -> unconnected-(U1-Pad33)
- U1 pad 34: no_connect_94 -> unconnected-(U1-Pad34)
- U1 pad 38: no_connect_95 -> unconnected-(U1-Pad38)
- U2 pad 10: no_connect_96 -> unconnected-(U2-Pad10)
- U2 pad 11: Net-(U2-Pad11) -> unconnected-(U2-Pad11)
- U2 pad 12: Net-(U2-Pad12) -> unconnected-(U2-Pad12)
- U2 pad 14: Net-(U2-Pad14) -> unconnected-(U2-Pad14)
- U2 pad 15: Net-(U2-Pad15) -> unconnected-(U2-Pad15)
- U2 pad 17: no_connect_97 -> unconnected-(U2-Pad17)
- U2 pad 18: no_connect_98 -> unconnected-(U2-Pad18)
- U2 pad 19: no_connect_99 -> unconnected-(U2-Pad19)
- U2 pad 2: Net-(U2-Pad2) -> unconnected-(U2-Pad2)
- U2 pad 3: Net-(U2-Pad3) -> unconnected-(U2-Pad3)
- U2 pad 4: Net-(U2-Pad4) -> unconnected-(U2-Pad4)
- U2 pad 6: no_connect_100 -> unconnected-(U2-Pad6)
- U2 pad 7: no_connect_101 -> unconnected-(U2-Pad7)
- U3 pad 6: no_connect_102 -> unconnected-(U3-Pad6)
- U4 pad 6: no_connect_103 -> unconnected-(U4-Pad6)
- U5 pad 6: no_connect_104 -> unconnected-(U5-Pad6)
