File: syzygy-sgmii/kicad-src/syzygy-sgmii.kicad_sch (KiCad schematic)
At the start: 90 parts, among them CON1 JD1_0001NL, J1 SYZYGY-TXR-4, U1 DP83867C, U3 TLV62569DRL, U4 TLV62569DRL, U5 TLV62569DRL, Y1 25MHz

Commit message: Finish syzygy-sgmii
Parts:
- removed TP5: TestPoint_Alt, TestPoint:TestPoint_Pad_D1.0mm, symbol Connector:TestPoint_Alt
- added C32: 0.1uF, Capacitor_SMD:C_0402_1005Metric, symbol Device:C
- added R16: 100R, Resistor_SMD:R_0402_1005Metric, symbol Device:R
- added R17: 10k, Resistor_SMD:R_0402_1005Metric, symbol Device:R
- added R18: 2.49k, Resistor_SMD:R_0402_1005Metric, symbol Device:R
- added U6, U7: TPD4EUSB30, Package_SON:USON-10_2.5x1.0mm_P0.5mm, symbol Power_Protection:TPD4EUSB30
- added X1: SG3225VAN, Oscillator:Oscillator_SMD_Silicon_Labs_LGA-6_2.5x3.2mm_P1.25mm, symbol gsd-kicad:SG3225VAN
Connections:
- net +3V3: now also C32.1, X1.1 (OE), X1.6 (Vcc)
- net ETH_A_N: now also U6.2 (D1-)
- net ETH_A_P: now also U6.1 (D1+)
- net ETH_B_N: now also U6.5 (D2-)
- net ETH_B_P: now also U6.4 (D2+)
- net ETH_C_N: now also U7.2 (D1-)
- net ETH_C_P: now also U7.1 (D1+)
- net ETH_D_N: now also U7.5 (D2-)
- net ETH_D_P: now also U7.4 (D2+)
- net GND: now also U1.25 (TX_D3), U1.26 (TX_D2), U1.29 (GTX_CLK), U1.37 (TX_CTRL), C32.2, R18.2, U6.3 (GND), U6.8 (GND), U7.3 (GND), U7.8 (GND), X1.3 (GND)
- net LED0: now also R17.1, R18.1
- net REFCLK_N: now also R16.1, X1.5 (~OUT)
- net REFCLK_P: now also R16.2, X1.4 (OUT)
- net VCCIO: now also R17.2
- net SGMII_SIN_N renamed SGMII_SI_N
- net SGMII_SIN_P renamed SGMII_SI_P
- net SGMII_SON_N renamed SGMII_SO_N
- net SGMII_SON_P renamed SGMII_SO_P
- net _SGMII_SIN_N renamed _SGMII_SI_N
- net _SGMII_SIN_P renamed _SGMII_SI_P
- net _SGMII_SON_N renamed _SGMII_SO_N
- net _SGMII_SON_P renamed _SGMII_SO_P
- no-connect marks 9 -> 5
Other:
- title: SYZYGY PCIe x4 -> SYZYGY SGMII
- moved on the sheet: D1, D2, D3, R12, R13, R14

Commit message: syzygy-sgmii: Add BOM values to project
Parts:
- C1, C2, C6, C7: Mfg (none) -> Yageo; PN (none) -> CC0402JRX7R7BB104
- C11, C5, C8: PN CC0402KRX5R6BB475 -> CC0402MRX5R5BB475
- C12, C13, C14: PN CC0402CRNPO9BN6R8 -> CC0402BRNPO9BN6R8
- C18, C19, C20: PN CC0402KRX5R6BB105 -> CC0402KRX5R8BB105
- C21, C22, C23, C24, C25, C26, C27, C28, C29, C30, C31, C32: PN CC0402KRX5R6BB105 -> CC0402JRX7R7BB104
- C3, C4: Mfg (none) -> Yageo; PN (none) -> CC0402JRNPO9BN100
- D1, D2, D3: Mfg (none) -> EKINGLUX; PN (none) -> E6C0603URAC1UDA
- J1: Mfg (none) -> Samtec Inc.; PN (none) -> QTH-020-01-F-D-DP-A-K
- R1: Mfg (none) -> Yageo; PN (none) -> AC0402FR-0711KL
- R10, R11, R12, R13, R14, R8, R9: Mfg (none) -> Yageo; PN (none) -> AC0402FR-071K5L
- R16: PN RC0402FR-07100KL -> AC0402FR-07100RL
- R17: Mfg (none) -> Yageo; PN (none) -> AC0402FR-0710KL
- R18: Mfg (none) -> Yageo; PN (none) -> AC0402FR-072K49L
- R2: value 84k5 -> 10K; PN RC0402FR-0784K5L -> AC0402FR-0710KL; Tol 1% -> (none)
- R3, R5: value 100k -> 15K; PN RC0402FR-07100KL -> AC0402FR-0715KL; Tol 1% -> (none)
- R4: value 84k5 -> 47.5K; PN RC0402FR-0784K5L -> AC0402FR-0747K5L; Tol 1% -> (none)
- R6: value 84k5 -> 20K; PN RC0402FR-0784K5L -> AC0402FR-0720KL; Tol 1% -> (none)
- R7: value 100k -> 10K; PN RC0402FR-07100KL -> AC0402FR-0710KL; Tol 1% -> (none)
- U1: Mfg (none) -> Texas Instruments; PN (none) -> DP83867CRRGZR
- U6, U7: Mfg (none) -> Texas Instruments; PN (none) -> TPD4EUSB30
- X1: Mfg (none) -> EPSON; PN (none) -> SG3225VEN 125.000000M-CJGA3
- Y1: Mfg (none) -> TAITIEN Elec; PN (none) -> XXDBCLNAOF-25.000000MHZ
