File: ecpbreaker/kicad-src/fpga.kicad_sch (KiCad schematic)
At the start: 28 parts, among them U11 TLV718P, U4 TLV62569DRL, U5 TLV62569DRL, U6 TLV725P, U8 ECP5U-12-CABGA256

Commit message: ecpbreaker: Add BOM values to project
Parts:
- C15, C23, C51: PN CC0402KRX5R6BB475 -> CC0402MRX5R5BB475
- C25, C30, C31, C43: PN CC0402KRX5R6BB105 -> CC0402KRX5R8BB105
- C26, C27: PN CC0402CRNPO9BN6R8 -> CC0402BRNPO9BN6R8
- C35, C36, C37, C38: PN CC0402KRX5R6BB105 -> CC0402JRX7R7BB104
- R10: value 210k -> 210K; PN RC0402FR-07210KL -> AC0402FR-07210KL; Tol 1% -> (none)
- R23: PN RC0402FR-0747KL -> AC0402FR-0747KL
- R24: PN RC0402FR-0784K5L -> AC0402FR-0784K5L; Tol 1% -> (none)
- R26: PN RC0402FR-07100KL -> AC0402FR-07100KL; Tol 1% -> (none)
- U11: PN TLV73318PDQNT -> TLV73318PDQNR
- U6: PN TLV73325PDQNT -> TLV74225PDQNR
- U8: PN (none) -> LFE5U-12F-7BG256I; manf# ECP5U_12 -> (none)
