File: ecpbreaker/kicad-src/pmods.kicad_sch (KiCad schematic)
At the start: 16 parts, among them J21 PMOD, J22 5V AUX, J23 PMOD, J26 5V AUX, J27 PMOD, U8 ECP5U-12-CABGA256

Commit message: ecpbreaker: Add BOM values to project
Parts:
- C32, C33, C34: DNP YES -> (none); Key cap-cer-0603-10u -> (none); Source ANY -> (none)
- C5: Mfg (none) -> Yageo; PN (none) -> CC0402JRX7R7BB104
- J21, J23, J27: Key conn-th-01in-6-2-rec-ra -> (none); Mfg (none) -> CJT(Changjiang Connectors); PN (none) -> A2541HWR-2x6P; Source ANY -> (none)
- J22, J26: Key conn-th-01in-2-1-hdr -> (none); Source ANY -> (none)
- R16, R17, R18, R3, R4, R7: Mfg (none) -> Yageo; PN (none) -> YC124-JR-0733RL
- U8: PN (none) -> LFE5U-12F-7BG256I; manf# ECP5U_12 -> (none)
