File: ecpbreaker/kicad-src/ram.kicad_sch (KiCad schematic)
At the start: 12 parts, among them U3 W25Q32JVSS, U8 ECP5U-12-CABGA256, U9 IS66WVH16M8ALL

Commit message: ecpbreaker: Add BOM values to project
Parts:
- C11, C20, C21, C3, C41: Mfg (none) -> Yageo; PN (none) -> CC0402JRX7R7BB104
- C22: value 100n -> 0.1uF; Key cap-cer-0402-100n -> (none); Mfg (none) -> Yageo; PN (none) -> CC0402JRX7R7BB104; Source ANY -> (none)
- R11: Mfg (none) -> Yageo; PN (none) -> YC124-JR-0710KL
- R19, R29: value 10k -> 10K; Key res-0402-10k -> (none); Mfg (none) -> Yageo; PN (none) -> AC0402FR-0710KL; Source ANY -> (none)
- U3: value W25Q32JVSS -> W25Q256; Mfg (none) -> Winbond Elec; PN (none) -> W25Q256JVEIQ
- U8: PN (none) -> LFE5U-12F-7BG256I; manf# ECP5U_12 -> (none)
Connections:
- net DONE renamed FPGA_DONE
- net PROGRAMn renamed ~FPGA_RESET
