File: ecpbreaker/kicad-src/syzygy.kicad_sch (KiCad schematic)
At the start: 16 parts, among them J1 SYZYGY-STD, U12 DAC081C081CIMK, U13 TPS73101DBV, U8 ECP5U-12-CABGA256

Commit message: ecpbreaker: Add BOM values to project
Parts:
- C44, C46: Mfg Samsung Electro-Mechanics -> Yageo; PN CL10A475KP8NNNC -> CC0603KRX5R6BB475
- C45, C47: value 100nF -> 0.1uF; Mfg Samsung Electro-Mechanics -> Yageo; PN CL05B104KP5NNNC -> CC0402JRX7R7BB104
- C8: Mfg (none) -> Yageo; PN (none) -> CC0402JRX7R7BB104
- R32: footprint Capacitor_SMD:C_0402_1005Metric -> Resistor_SMD:R_0402_1005Metric; Mfg Stackpole Electronics Inc -> Yageo; PN RNCF0402DTE10K0 -> AC0402FR-0710KL; Tol 1% -> (none)
- R33: footprint Capacitor_SMD:C_0402_1005Metric -> Resistor_SMD:R_0402_1005Metric; Mfg Stackpole Electronics Inc -> Yageo; PN RNCF0402DTE33K0 -> AC0402FR-0733KL; Tol 0.5% -> (none)
- R34: footprint Capacitor_SMD:C_0402_1005Metric -> Resistor_SMD:R_0402_1005Metric; Mfg Stackpole Electronics Inc -> Yageo; PN RNCF0402DTE24K9 -> AC0402FR-0724K9L; Tol 0.5% -> (none)
- R35: value R -> 210K; Mfg (none) -> Yageo; PN (none) -> AC0402FR-07210KL
- R8: footprint Capacitor_SMD:C_0402_1005Metric -> Resistor_SMD:R_0402_1005Metric; Mfg Stackpole Electronics Inc -> Yageo; PN RNCF0402DTE42K2 -> AC0402FR-0742K2L; Tol 0.5% -> (none)
- U8: PN (none) -> LFE5U-12F-7BG256I; manf# ECP5U_12 -> (none)
