File: gpdi/kicad-src/gpdi-sink.kicad_sch (KiCad schematic)
At the start: 32 parts, among them J5 GPDI_A_1.4

Commit message: syzygy-gpdi: Add BOM values to project
Parts:
- C11, C13, C14, C15, C16, C17, C18, C19, C20: value 0.1u -> 0.1uF; Mfg (none) -> Yageo; PN (none) -> CC0402JRX7R7BB104
- C12: value 4.7u -> 4.7uF; Mfg (none) -> Yageo; PN (none) -> CC0402MRX5R5BB475
- J5: Mfg (none) -> Amphenol ICC (FCI); PN (none) -> 10029449-111RLF
- R10, R13, R14, R18, R19, R20, R21, R22: Mfg (none) -> Yageo; PN (none) -> AC0402FR-0751RL
- R2: Mfg (none) -> Yageo; PN (none) -> AC0402FR-072KL
- R3, R9: Mfg (none) -> Yageo; PN (none) -> AC0402FR-071KL
- R4, R5, R7, R8: Mfg (none) -> Yageo; PN (none) -> AC0402FR-0747KL
