File: gpdi/kicad-src/gpdi-source.kicad_sch (KiCad schematic)
At the start: 16 parts, among them J2 GPDI_A_1.4

Commit message: syzygy-gpdi: Add BOM values to project
Parts:
- C1, C2, C3, C4, C5, C6, C7, C8: value 0.1u -> 0.1uF; Mfg (none) -> Yageo; PN (none) -> CC0402JRX7R7BB104
- J2: Mfg (none) -> Amphenol ICC (FCI); PN (none) -> 10029449-111RLF
- R1: Mfg (none) -> Yageo; PN (none) -> AC0402FR-071KL
- R23: Mfg (none) -> Yageo; PN (none) -> AC0402FR-070RL
Changed lines of the file:
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@@
-(kicad_sch (version 20201015) (generator eeschema)
-  (page 1 4)
+(kicad_sch (version 20210126) (generator eeschema)
   (paper "A4")
   (title_block
@@
       (effects (font (size 1.27 1.27)) hide)
     )
+    (pin "1")
   )
   (symbol (lib_id "Connector:TestPoint") (at 194.31 109.22 90) (unit 1)
@@
       (effects (font (size 1.27 1.27)) hide)
     )
+    (pin "1")
   )
   (symbol (lib_id "Connector:TestPoint") (at 194.31 114.3 90) (unit 1)
@@
       (effects (font (size 1.27 1.27)) hide)
     )
+    (pin "1")
   )
   (symbol (lib_id "Connector:TestPoint") (at 194.31 116.84 90) (unit 1)
@@
       (effects (font (size 1.27 1.27)) hide)
     )
+    (pin "1")
   )
   (symbol (lib_id "Connector:TestPoint") (at 194.31 121.92 90) (unit 1)
@@
       (effects (font (size 1.27 1.27)) hide)
     )
+    (pin "1")
   )
   (symbol (lib_id "power:+5V") (at 196.85 53.34 0) (unit 1)
@@
       (effects (font (size 1.27 1.27)) hide)
     )
+    (pin "1")
   )
   (symbol (lib_id "power:GND") (at 209.55 139.7 0) (unit 1)
@@
       (effects (font (size 1.27 1.27)) hide)
     )
+    (pin "1")
   )
   (symbol (lib_id "Device:R") (at 180.34 119.38 0) (unit 1)
@@
       (effects (font (size 1.27 1.27)) hide)
     )
+    (property "Mfg" "Yageo" (id 4) (at 180.34 119.38 0)
+      (effects (font (size 1.27 1.27)) hide)
+    )
+    (property "PN" "AC0402FR-071KL" (id 5) (at 180.34 119.38 0)
+      (effects (font (size 1.27 1.27)) hide)
+    )
+    (pin "1")
+    (pin "2")
   )
   (symbol (lib_id "Device:R") (at 196.85 57.15 0) (unit 1)
@@
       (effects (font (size 1.27 1.27)) hide)
     )
+    (property "Mfg" "Yageo" (id 4) (at 196.85 57.15 0)
+      (effects (font (size 1.27 1.27)) hide)
+    )
+    (property "PN" "AC0402FR-070RL" (id 5) (at 196.85 57.15 0)
+      (effects (font (size 1.27 1.27)) hide)
+    )
+    (pin "1")
+    (pin "2")
   )
   (symbol (lib_id "Device:C") (at 157.48 88.9 90) (unit 1)
@@
       (effects (font (size 1.27 1.27)) hide)
     )
-    (property "Value" "0.1u" (id 1) (at 157.48 83.82 90)
+    (property "Value" "0.1uF" (id 1) (at 157.48 83.82 90)
       (effects (font (size 1.27 1.27)) hide)
     )
@@
       (effects (font (size 1.27 1.27)) hide)
     )
+    (property "Mfg" "Yageo" (id 4) (at 157.48 88.9 0)
+      (effects (font (size 1.27 1.27)) hide)
+    )
+    (property "PN" "CC0402JRX7R7BB104" (id 5) (at 157.48 88.9 0)
+      (effects (font (size 1.27 1.27)) hide)
+    )
+    (pin "1")
+    (pin "2")
   )
   (symbol (lib_id "Device:C") (at 157.48 93.98 90) (unit 1)
@@
       (effects (font (size 1.27 1.27)) hide)
     )
-    (property "Value" "0.1u" (id 1) (at 157.48 88.9 90)
+    (property "Value" "0.1uF" (id 1) (at 157.48 88.9 90)
       (effects (font (size 1.27 1.27)) hide)
     )
@@
       (effects (font (size 1.27 1.27)) hide)
     )
+    (property "Mfg" "Yageo" (id 4) (at 157.48 93.98 0)
+      (effects (font (size 1.27 1.27)) hide)
+    )
+    (property "PN" "CC0402JRX7R7BB104" (id 5) (at 157.48 93.98 0)
+      (effects (font (size 1.27 1.27)) hide)
+    )
+    (pin "1")
+    (pin "2")
   )
   (symbol (lib_id "Device:C") (at 157.48 99.06 90) (unit 1)
@@
       (effects (font (size 1.27 1.27)) hide)
     )
-    (property "Value" "0.1u" (id 1) (at 157.48 93.98 90)
+    (property "Value" "0.1uF" (id 1) (at 157.48 93.98 90)
       (effects (font (size 1.27 1.27)) hide)
     )
@@
       (effects (font (size 1.27 1.27)) hide)
     )
+    (property "Mfg" "Yageo" (id 4) (at 157.48 99.06 0)
+      (effects (font (size 1.27 1.27)) hide)
+    )
+    (property "PN" "CC0402JRX7R7BB104" (id 5) (at 157.48 99.06 0)
+      (effects (font (size 1.27 1.27)) hide)
+    )
+    (pin "1")
+    (pin "2")
   )
   (symbol (lib_id "Device:C") (at 157.48 104.14 90) (unit 1)
@@
       (effects (font (size 1.27 1.27)) hide)
     )
-    (property "Value" "0.1u" (id 1) (at 157.48 99.06 90)
+    (property "Value" "0.1uF" (id 1) (at 157.48 99.06 90)
       (effects (font (size 1.27 1.27)) hide)
     )
@@
       (effects (font (size 1.27 1.27)) hide)
     )
+    (property "Mfg" "Yageo" (id 4) (at 157.48 104.14 0)
+      (effects (font (size 1.27 1.27)) hide)
+    )
+    (property "PN" "CC0402JRX7R7BB104" (id 5) (at 157.48 104.14 0)
+      (effects (font (size 1.27 1.27)) hide)
+    )
+    (pin "1")
+    (pin "2")
   )
   (symbol (lib_id "Device:C") (at 163.83 86.36 90) (unit 1)
@@
       (effects (font (size 1.27 1.27)) hide)
     )
-    (property "Value" "0.1u" (id 1) (at 163.83 81.28 90)
+    (property "Value" "0.1uF" (id 1) (at 163.83 81.28 90)
       (effects (font (size 1.27 1.27)) hide)
     )
@@
       (effects (font (size 1.27 1.27)) hide)
     )
+    (property "Mfg" "Yageo" (id 4) (at 163.83 86.36 0)
+      (effects (font (size 1.27 1.27)) hide)
+    )
+    (property "PN" "CC0402JRX7R7BB104" (id 5) (at 163.83 86.36 0)
+      (effects (font (size 1.27 1.27)) hide)
+    )
+    (pin "1")
+    (pin "2")
   )
   (symbol (lib_id "Device:C") (at 163.83 91.44 90) (unit 1)
@@
       (effects (font (size 1.27 1.27)) hide)
     )
-    (property "Value" "0.1u" (id 1) (at 163.83 86.36 90)
+    (property "Value" "0.1uF" (id 1) (at 163.83 86.36 90)
       (effects (font (size 1.27 1.27)) hide)
     )
@@
       (effects (font (size 1.27 1.27)) hide)
     )
+    (property "Mfg" "Yageo" (id 4) (at 163.83 91.44 0)
+      (effects (font (size 1.27 1.27)) hide)
+    )
+    (property "PN" "CC0402JRX7R7BB104" (id 5) (at 163.83 91.44 0)
+      (effects (font (size 1.27 1.27)) hide)
+    )
+    (pin "1")
+    (pin "2")
   )
   (symbol (lib_id "Device:C") (at 163.83 96.52 90) (unit 1)
@@
       (effects (font (size 1.27 1.27)) hide)
     )
-    (property "Value" "0.1u" (id 1) (at 163.83 91.44 90)
+    (property "Value" "0.1uF" (id 1) (at 163.83 91.44 90)
       (effects (font (size 1.27 1.27)) hide)
     )
@@
       (effects (font (size 1.27 1.27)) hide)
     )
+    (property "Mfg" "Yageo" (id 4) (at 163.83 96.52 0)
+      (effects (font (size 1.27 1.27)) hide)
+    )
+    (property "PN" "CC0402JRX7R7BB104" (id 5) (at 163.83 96.52 0)
+      (effects (font (size 1.27 1.27)) hide)
+    )
+    (pin "1")
+    (pin "2")
   )
   (symbol (lib_id "Device:C") (at 163.83 101.6 90) (unit 1)
@@
       (effects (font (size 1.27 1.27)) hide)
     )
-    (property "Value" "0.1u" (id 1) (at 163.83 96.52 90)
+    (property "Value" "0.1uF" (id 1) (at 163.83 96.52 90)
       (effects (font (size 1.27 1.27)) hide)
     )
@@
       (effects (font (size 1.27 1.27)) hide)
     )
+    (property "Mfg" "Yageo" (id 4) (at 163.83 101.6 0)
+      (effects (font (size 1.27 1.27)) hide)
+    )
+    (property "PN" "CC0402JRX7R7BB104" (id 5) (at 163.83 101.6 0)
+      (effects (font (size 1.27 1.27)) hide)
+    )
+    (pin "1")
+    (pin "2")
   )
   (symbol (lib_id "Connector:HDMI_A_1.4") (at 214.63 106.68 0) (unit 1)
@@
       (effects (font (size 1.27 1.27)) hide)
     )
-    (property "Datasheet" "https://en.wikipedia.org/wiki/HDMI" (id 3) (at 215.265 106.68 0)
-      (effects (font (size 1.27 1.27)) hide)
-    )
+    (property "Datasheet" "" (id 3) (at 215.265 106.68 0)
+      (effects (font (size 1.27 1.27)) hide)
+    )
+    (property "Mfg" "Amphenol ICC (FCI)" (id 4) (at 214.63 106.68 0)
+      (effects (font (size 1.27 1.27)) hide)
+    )
+    (property "PN" "10029449-111RLF" (id 5) (at 214.63 106.68 0)
+      (effects (font (size 1.27 1.27)) hide)
+    )
+    (pin "1")
+    (pin "10")
+    (pin "11")
+    (pin "12")
+    (pin "13")
+    (pin "14")
+    (pin "15")
+    (pin "16")
+    (pin "17")
+    (pin "18")
+    (pin "19")
+    (pin "2")
+    (pin "3")
+    (pin "4")
+    (pin "5")
+    (pin "6")
+    (pin "7")
+    (pin "8")
+    (pin "9")
+    (pin "SH")
   )
 )
