File: gpdi/kicad-src/gpdi.kicad_pcb (KiCad board)
At the start: 4 copper layers, 45 x 35 mm, 65 parts, among them J1 SYZYGY-STD, J2 GPDI_A_1.4, J3 TagConnect, J4 Conn_01x03_Male, J5 GPDI_A_1.4, U2 ATtiny44A-MMH

Commit message: syzygy-gpdi: Add BOM values to project
Parts:
- C1, C11, C13, C14, C15, C16, C17, C18, C19, C2, C20, C3, C4, C5, C6, C7, C8: value 0.1u -> 0.1uF
- C12: value 4.7u -> 4.7uF
Connections:
- J1 pad 18: Net-(J1-Pad18) -> unconnected-(J1-Pad18)
- J1 pad 20: Net-(J1-Pad20) -> unconnected-(J1-Pad20)
- J1 pad 22: Net-(J1-Pad22) -> unconnected-(J1-Pad22)
- J1 pad 24: Net-(J1-Pad24) -> unconnected-(J1-Pad24)
- J1 pad 26: Net-(J1-Pad26) -> unconnected-(J1-Pad26)
- J1 pad 27: Net-(J1-Pad27) -> unconnected-(J1-Pad27)
- J1 pad 28: Net-(J1-Pad28) -> unconnected-(J1-Pad28)
- J1 pad 29: Net-(J1-Pad29) -> unconnected-(J1-Pad29)
- J1 pad 30: Net-(J1-Pad30) -> unconnected-(J1-Pad30)
- J1 pad 31: Net-(J1-Pad31) -> unconnected-(J1-Pad31)
- J1 pad 32: Net-(J1-Pad32) -> unconnected-(J1-Pad32)
- J1 pad 37: Net-(J1-Pad37) -> unconnected-(J1-Pad37)
- J1 pad 38: Net-(J1-Pad38) -> unconnected-(J1-Pad38)
- U2 pad 10: Net-(U2-Pad10) -> unconnected-(U2-Pad10)
- U2 pad 11: Net-(U2-Pad11) -> unconnected-(U2-Pad11)
- U2 pad 12: Net-(U2-Pad12) -> unconnected-(U2-Pad12)
- U2 pad 14: Net-(U2-Pad14) -> unconnected-(U2-Pad14)
- U2 pad 15: Net-(U2-Pad15) -> unconnected-(U2-Pad15)
- U2 pad 17: Net-(U2-Pad17) -> unconnected-(U2-Pad17)
- U2 pad 18: Net-(U2-Pad18) -> unconnected-(U2-Pad18)
- U2 pad 19: Net-(U2-Pad19) -> unconnected-(U2-Pad19)
- U2 pad 2: Net-(U2-Pad2) -> unconnected-(U2-Pad2)
- U2 pad 3: Net-(U2-Pad3) -> unconnected-(U2-Pad3)
- U2 pad 4: Net-(U2-Pad4) -> unconnected-(U2-Pad4)
- U2 pad 6: Net-(U2-Pad6) -> unconnected-(U2-Pad6)
- U2 pad 7: Net-(U2-Pad7) -> unconnected-(U2-Pad7)
