File: gpdi/kicad-src/gpdi.kicad_sch (KiCad schematic)
At the start: 10 parts, among them J1 SYZYGY-STD, J4 Conn_01x03_Male

Commit message: syzygy-gpdi: Add BOM values to project
Parts:
- D2, D3, D4: Mfg (none) -> TOGIALED; PN (none) -> TJ-S1005SW4TGLC7K-A5
- R11, R12, R16, R17, R6: Mfg (none) -> Yageo; PN (none) -> AC0402FR-071KL
