File: syzygy-epc901/kicad-src/epc901.kicad_sch (KiCad schematic)
At the start: 43 parts, among them U3 EPC901

Commit message: syzygy-epc901: Add BOM values to project
Parts:
- C11: Mfg (none) -> Yageo; PN (none) -> CC0402JRX7R7BB104
- C13, C6, C7: Mfg (none) -> Yageo; PN (none) -> CC0402KRX5R8BB105
- C14, C15: Mfg (none) -> Yageo; PN (none) -> CC0402KRX5R6BB225
- C8: Mfg (none) -> Yageo; PN (none) -> CC0603KRX5R5BB106
- L1: Mfg (none) -> Murata Electronics; Mpn BLM18TG601TN1D -> (none); PN (none) -> BLM15HG601SN1D
- R10, R9: Mfg (none) -> Yageo; PN (none) -> AC0402FR-072K2L
- R22: Mfg (none) -> Yageo; PN (none) -> AC0402FR-0756KL
- R23, R24, R25, R32: Mfg (none) -> Yageo; PN (none) -> AC0402FR-070RL
- U3: Mfg (none) -> ESPROS Photonics AG; Mpn EPC901-CSP32-033 -> (none); PN (none) -> EPC901-CSP32-033
- gave numbers to parts that had none: 1
