File: syzygy-epc901/kicad-src/syzygy-epc901.kicad_pcb (KiCad board)
At the start: 4 copper layers, 45 x 70 mm, 113 parts, among them J1 SYZYGY-STD, J2 Conn_01x02_Male, J3 TagConnect, J4 Conn_01x02_Male, J5 Conn_01x02_Male, J6 Conn_01x02_Male, U1 AD9629, U2 ATtiny44A-MMH, U3 EPC901, U4 LT1962-1.8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

Commit message: syzygy-epc901: Add BOM values to project
Connections:
- net GNDA renamed GND
- J1 pad 16: no_connect_107 -> unconnected-(J1-Pad16)
- J1 pad 37: Net-(J1-Pad37) -> unconnected-(J1-Pad37)
- J1 pad 38: Net-(J1-Pad38) -> unconnected-(J1-Pad38)
- U2 pad 10: (no net) -> unconnected-(U2-Pad10)
- U2 pad 11: Net-(U2-Pad11) -> unconnected-(U2-Pad11)
- U2 pad 12: Net-(U2-Pad12) -> unconnected-(U2-Pad12)
- U2 pad 14: Net-(U2-Pad14) -> unconnected-(U2-Pad14)
- U2 pad 15: Net-(U2-Pad15) -> unconnected-(U2-Pad15)
- U2 pad 17: (no net) -> unconnected-(U2-Pad17)
- U2 pad 18: (no net) -> unconnected-(U2-Pad18)
- U2 pad 19: (no net) -> unconnected-(U2-Pad19)
- U2 pad 2: Net-(U2-Pad2) -> unconnected-(U2-Pad2)
- U2 pad 3: Net-(U2-Pad3) -> unconnected-(U2-Pad3)
- U2 pad 4: Net-(U2-Pad4) -> unconnected-(U2-Pad4)
- U2 pad 6: (no net) -> unconnected-(U2-Pad6)
- U2 pad 7: (no net) -> unconnected-(U2-Pad7)
- U4 pad 6: (no net) -> unconnected-(U4-Pad6)
- U4 pad 7: (no net) -> unconnected-(U4-Pad7)
Routing:
- net unconnected-(J1-Pad16): track 0.00 -> 2.20 mm, vias 0 -> 1
- net no_connect_107: track 2.20 -> 0.00 mm, vias 1 -> 0
