File: syzygy-epc901/kicad-src/syzygy-epc901.kicad_sch (KiCad schematic)
At the start: 62 parts, among them J1 SYZYGY-STD, J2 Conn_01x02_Male, J4 Conn_01x02_Male, J5 Conn_01x02_Male, J6 Conn_01x02_Male, U1 AD9629, U4 LT1962-1.8, U5 TLP291, U6 TLP291, U7 TLP291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

Commit message: syzygy-epc901: Add BOM values to project
Parts:
- C1, C20, C21, C22, C23, C24, C26, C4, C5: Mfg (none) -> Yageo; PN (none) -> CC0402JRX7R7BB104
- C16, C19, C2, C25: Mfg (none) -> Yageo; PN (none) -> CC0402KRX5R8BB105
- C17: Mfg (none) -> Yageo; PN (none) -> CC0402JRX7R9BB103
- C18: Mfg (none) -> Yageo; PN (none) -> CC0603KRX5R5BB106
- C3: Mfg (none) -> Yageo; PN (none) -> CC0402JRNPO9BN220
- J1: PN QTE-020-01-F-D-A -> QTE-020-01-F-D-A-K
- R2: Mfg (none) -> Yageo; PN (none) -> AC0402FR-070RL
- R3, R4: Mfg (none) -> Yageo; PN (none) -> AC0402FR-0733RL
- R33, R34: Mfg (none) -> Yageo; PN (none) -> AC0402FR-071KL
- R35, R36, R37, R38, R39, R40, R41, R42, R43, R44, R45, R46, R47, R48, R5, R52, R53, R54, R55, R6, R7, R8: Mfg (none) -> Yageo; PN (none) -> AC0402FR-07100RL
- R49: Mfg (none) -> Yageo; PN (none) -> AC0402FR-0710KL
- R50, R51: Mfg (none) -> Yageo; PN (none) -> AC0402FR-072K2L
- U1: Mfg (none) -> Analog Devices Inc.; PN (none) -> AD9629BCPZ-65
- U4: Mfg (none) -> Analog Devices Inc.; PN (none) -> LT1962EMS8-1.8#PBF
- U5, U6, U7, U8: Mfg (none) -> TOSHIBA; PN (none) -> TLP291(GB-TP,SE
