File: icebreaker++-ram/kicad-src/fpga.kicad_sch (KiCad schematic)
At the start: 24 parts, among them U4 TLV62569DRL, U5 TLV62569DRL, U6 TLV713285PDBV, U8 ECP5U-12-CABGA256

Commit message: icebreaker++ram: Add BOM values to project
Parts:
- C15, C23: Mfg Yageo -> TDK; PN CC0402KRX5R6BB475 -> C1005X5R0J475K050BE
- C35, C36, C37, C38: Mfg Yageo -> KEMET; PN CC0402KRX5R6BB105 -> C0402C104K8PAC7411
- L3, L4: Mfg Sunltech Tech -> (none); PN SLM20122R2MIT -> (none)
- R10, R23, R24, R26: Mfg Yageo -> (none)
- U4, U5: Mfg Texas Instruments -> (none)
- U6: PN (none) -> TLV713285PDBVR
- U8: PN (none) -> LFE5U-12F-8BG256C
Changed lines of the file:
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@@
       (effects (font (size 1.27 1.27)) hide)
     )
-    (property "Mfg" "Sunltech Tech" (id 4) (at 72.39 76.2 0)
-      (effects (font (size 1.27 1.27)) hide)
-    )
-    (property "PN" "SLM20122R2MIT" (id 5) (at 72.39 76.2 0)
+    (property "Mfg" "" (id 4) (at 72.39 76.2 0)
+      (effects (font (size 1.27 1.27)) hide)
+    )
+    (property "PN" "" (id 5) (at 72.39 76.2 0)
       (effects (font (size 1.27 1.27)) hide)
     )
@@
       (effects (font (size 1.27 1.27)) hide)
     )
-    (property "Mfg" "Sunltech Tech" (id 4) (at 72.39 123.19 0)
-      (effects (font (size 1.27 1.27)) hide)
-    )
-    (property "PN" "SLM20122R2MIT" (id 5) (at 72.39 123.19 0)
+    (property "Mfg" "" (id 4) (at 72.39 123.19 0)
+      (effects (font (size 1.27 1.27)) hide)
+    )
+    (property "PN" "" (id 5) (at 72.39 123.19 0)
       (effects (font (size 1.27 1.27)) hide)
     )
@@
       (effects (font (size 1.27 1.27)) hide)
     )
-    (property "Mfg" "Yageo" (id 5) (at 77.47 82.55 0)
+    (property "Mfg" "" (id 5) (at 77.47 82.55 0)
       (effects (font (size 1.27 1.27)) hide)
     )
@@
       (effects (font (size 1.27 1.27)) hide)
     )
-    (property "Mfg" "Yageo" (id 5) (at 77.47 95.25 0)
+    (property "Mfg" "" (id 5) (at 77.47 95.25 0)
       (effects (font (size 1.27 1.27)) hide)
     )
@@
       (effects (font (size 1.27 1.27)) hide)
     )
-    (property "Mfg" "Yageo" (id 5) (at 77.47 129.54 0)
+    (property "Mfg" "" (id 5) (at 77.47 129.54 0)
       (effects (font (size 1.27 1.27)) hide)
     )
@@
       (effects (font (size 1.27 1.27)) hide)
     )
-    (property "Mfg" "Yageo" (id 5) (at 77.47 142.24 0)
+    (property "Mfg" "" (id 5) (at 77.47 142.24 0)
       (effects (font (size 1.27 1.27)) hide)
     )
@@
       (effects (font (size 1.27 1.27)) hide)
     )
-    (property "Mfg" "Yageo" (id 4) (at 100.33 218.44 0)
-      (effects (font (size 1.27 1.27)) hide)
-    )
-    (property "PN" "CC0402KRX5R6BB475" (id 5) (at 100.33 218.44 0)
+    (property "Mfg" "TDK" (id 4) (at 100.33 218.44 0)
+      (effects (font (size 1.27 1.27)) hide)
+    )
+    (property "PN" "C1005X5R0J475K050BE" (id 5) (at 100.33 218.44 0)
       (effects (font (size 1.27 1.27)) hide)
     )
@@
       (effects (font (size 1.27 1.27)) hide)
     )
-    (property "Mfg" "Yageo" (id 4) (at 100.33 265.43 0)
-      (effects (font (size 1.27 1.27)) hide)
-    )
-    (property "PN" "CC0402KRX5R6BB475" (id 5) (at 100.33 265.43 0)
+    (property "Mfg" "TDK" (id 4) (at 100.33 265.43 0)
+      (effects (font (size 1.27 1.27)) hide)
+    )
+    (property "PN" "C1005X5R0J475K050BE" (id 5) (at 100.33 265.43 0)
       (effects (font (size 1.27 1.27)) hide)
     )
@@
       (effects (font (size 1.27 1.27)) hide)
     )
-    (property "Mfg" "Yageo" (id 4) (at 134.62 311.15 0)
-      (effects (font (size 1.27 1.27)) hide)
-    )
-    (property "PN" "CC0402KRX5R6BB105" (id 5) (at 134.62 311.15 0)
+    (property "Mfg" "KEMET" (id 4) (at 134.62 311.15 0)
+      (effects (font (size 1.27 1.27)) hide)
+    )
+    (property "PN" "C0402C104K8PAC7411" (id 5) (at 134.62 311.15 0)
       (effects (font (size 1.27 1.27)) hide)
     )
@@
       (effects (font (size 1.27 1.27)) hide)
     )
-    (property "Mfg" "Yageo" (id 4) (at 142.24 311.15 0)
-      (effects (font (size 1.27 1.27)) hide)
-    )
-    (property "PN" "CC0402KRX5R6BB105" (id 5) (at 142.24 311.15 0)
+    (property "Mfg" "KEMET" (id 4) (at 142.24 311.15 0)
+      (effects (font (size 1.27 1.27)) hide)
+    )
+    (property "PN" "C0402C104K8PAC7411" (id 5) (at 142.24 311.15 0)
       (effects (font (size 1.27 1.27)) hide)
     )
@@
       (effects (font (size 1.27 1.27)) hide)
     )
-    (property "Mfg" "Yageo" (id 4) (at 149.86 311.15 0)
-      (effects (font (size 1.27 1.27)) hide)
-    )
-    (property "PN" "CC0402KRX5R6BB105" (id 5) (at 149.86 311.15 0)
+    (property "Mfg" "KEMET" (id 4) (at 149.86 311.15 0)
+      (effects (font (size 1.27 1.27)) hide)
+    )
+    (property "PN" "C0402C104K8PAC7411" (id 5) (at 149.86 311.15 0)
       (effects (font (size 1.27 1.27)) hide)
     )
@@
       (effects (font (size 1.27 1.27)) hide)
     )
-    (property "Mfg" "Yageo" (id 4) (at 157.48 311.15 0)
-      (effects (font (size 1.27 1.27)) hide)
-    )
-    (property "PN" "CC0402KRX5R6BB105" (id 5) (at 157.48 311.15 0)
+    (property "Mfg" "KEMET" (id 4) (at 157.48 311.15 0)
+      (effects (font (size 1.27 1.27)) hide)
+    )
+    (property "PN" "C0402C104K8PAC7411" (id 5) (at 157.48 311.15 0)
       (effects (font (size 1.27 1.27)) hide)
     )
@@
       (effects (font (size 1.27 1.27)) hide)
     )
+    (property "PN" "TLV713285PDBVR" (id 4) (at 59.69 44.45 0)
+      (effects (font (size 1.27 1.27)) hide)
+    )
   )
   (symbol (lib_id "Regulator_Switching:TLV62569DRL") (at 58.42 81.28 0) (unit 1)
@@
       (effects (font (size 1.27 1.27)) hide)
     )
-    (property "Mfg" "Texas Instruments" (id 4) (at 58.42 81.28 0)
+    (property "Mfg" "" (id 4) (at 58.42 81.28 0)
       (effects (font (size 1.27 1.27)) hide)
     )
@@
       (effects (font (size 1.27 1.27)) hide)
     )
-    (property "Mfg" "Texas Instruments" (id 4) (at 58.42 128.27 0)
+    (property "Mfg" "" (id 4) (at 58.42 128.27 0)
       (effects (font (size 1.27 1.27)) hide)
     )
@@
       (effects (font (size 1.524 1.524)) (justify right) hide)
     )
+    (property "PN" "LFE5U-12F-8BG256C" (id 4) (at 193.04 144.78 0)
+      (effects (font (size 1.27 1.27)) hide)
+    )
   )
   (symbol (lib_id "gsd-kicad:ECP5U-12-CABGA256") (at 195.58 53.34 0) (unit 2)
@@
       (effects (font (size 1.524 1.524)) (justify right) hide)
     )
-  )
+    (property "PN" "LFE5U-12F-8BG256C" (id 4) (at 195.58 53.34 0)
+      (effects (font (size 1.27 1.27)) hide)
+    )
+  )
