File: icebreaker++-ram/kicad-src/icebreaker++.kicad_sch (KiCad schematic)
At the start: 58 parts, among them J20 Flash, J24 USB_C_Receptacle_USB2.0, J25 RGB Led, J28 CRESET, P2 UP, P3 UP, P4 UP, P5 UP, P6 RAM_CS, SW1 TACT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

Commit message: icebreaker++ram: Add BOM values to project
Parts:
- C1, C10, C12, C13, C14, C16, C17, C18, C19, C20, C21, C22, C4: value 100n -> 0.1uF; Mfg (none) -> KEMET; PN (none) -> C0402C104K8PAC7411
- C11, C2, C43: Mfg (none) -> KEMET; PN (none) -> C0402C104K8PAC7411
- D1, D4: Mfg (none) -> ROHM Semiconductor; PN (none) -> SML-D12P8WT86
- D11: Mfg (none) -> Cree, Inc.; PN (none) -> CLY6D-FKC-CNP1ST1E1BB7D3D3
- D3: Mfg (none) -> ROHM Semiconductor; PN (none) -> SMLD12BN1WT86
- D5: Mfg (none) -> ROHM Semiconductor; PN (none) -> SML-D12V8WT86
- R1: PN (none) -> MCS04020C1004FE000
- R11, R2: PN (none) -> EXB-28V103JX
- R12, R6: PN (none) -> RC0402FR-072K2L
- R13, R19, R25, R9: PN (none) -> RC0402FR-0710KL
- R14, R15, R5: PN (none) -> RC0402FR-07330RL
- R20: PN (none) -> RT0402FRE071KL
- R21, R22: PN (none) -> AF0402JR-075K1L
- R8: PN (none) -> RC0402FR-0712KL
- SW1: PN (none) -> PTS810SJK250SMTRLFS
- U1: PN (none) -> 93LC46BT-I/OT
- U2: Mfg (none) -> FTDI; PN (none) -> FT2232HQ-TRAY
- U3: PN (none) -> W25Q32JVSSIQ TR
- U7: PN (none) -> SIT2001BI-S2-33E-12.000000G
- U8: PN (none) -> LFE5U-12F-8BG256C
