File: icebreaker++-ram/kicad-src/pmods.kicad_sch (KiCad schematic)
At the start: 19 parts, among them J21 PMOD, J22 5V AUX, J23 PMOD, J26 5V AUX, J27 PMOD, U8 ECP5U-12-CABGA256, U9 LY68L6400SLIT

Commit message: icebreaker++ram: Add BOM values to project
Parts:
- C3, C39, C5: Mfg (none) -> KEMET; PN (none) -> C0402C104K8PAC7411
- U8: PN (none) -> LFE5U-12F-8BG256C
Changed lines of the file:
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@@
+      (effects (font (size 1.27 1.27)) hide)
+    )
+    (property "Mfg" "KEMET" (id 4) (at 24.13 114.3 0)
+      (effects (font (size 1.27 1.27)) hide)
+    )
+    (property "PN" "C0402C104K8PAC7411" (id 5) (at 24.13 114.3 0)
       (effects (font (size 1.27 1.27)) hide)
     )
@@
       (effects (font (size 1.27 1.27)) hide)
     )
+    (property "Mfg" "KEMET" (id 4) (at 29.21 22.86 0)
+      (effects (font (size 1.27 1.27)) hide)
+    )
+    (property "PN" "C0402C104K8PAC7411" (id 5) (at 29.21 22.86 0)
+      (effects (font (size 1.27 1.27)) hide)
+    )
   )
   (symbol (lib_id "Device:C") (at 123.19 151.13 270) (unit 1)
@@
     )
     (property "Datasheet" "~" (id 3) (at 123.19 151.13 0)
+      (effects (font (size 1.27 1.27)) hide)
+    )
+    (property "Mfg" "KEMET" (id 4) (at 123.19 151.13 0)
+      (effects (font (size 1.27 1.27)) hide)
+    )
+    (property "PN" "C0402C104K8PAC7411" (id 5) (at 123.19 151.13 0)
       (effects (font (size 1.27 1.27)) hide)
     )
@@
       (effects (font (size 1.524 1.524)) (justify right) hide)
     )
+    (property "PN" "LFE5U-12F-8BG256C" (id 4) (at 77.47 114.3 0)
+      (effects (font (size 1.27 1.27)) hide)
+    )
   )
   (symbol (lib_id "gsd-kicad:ECP5U-12-CABGA256") (at 82.55 22.86 0) (mirror y) (unit 7)
@@
       (effects (font (size 1.524 1.524)) (justify right) hide)
     )
+    (property "PN" "LFE5U-12F-8BG256C" (id 4) (at 82.55 22.86 0)
+      (effects (font (size 1.27 1.27)) hide)
+    )
   )
