File: icebreaker++-ram/kicad-src/ram.kicad_sch (KiCad schematic)
At the start: 6 parts, among them U10 IS66WVH16M8ALL, U8 ECP5U-12-CABGA256

Commit message: icebreaker++ram: Add BOM values to project
Parts:
- C40, C41, C42, C8: Mfg (none) -> KEMET; PN (none) -> C0402C104K8PAC7411
- U10: Mfg ISSI, Integrated Silicon Solution Inc -> (none)
- U8: PN (none) -> LFE5U-12F-8BG256C
Changed lines of the file:
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@@
+      (effects (font (size 1.27 1.27)) hide)
+    )
+    (property "Mfg" "KEMET" (id 4) (at 86.36 60.96 0)
+      (effects (font (size 1.27 1.27)) hide)
+    )
+    (property "PN" "C0402C104K8PAC7411" (id 5) (at 86.36 60.96 0)
       (effects (font (size 1.27 1.27)) hide)
     )
@@
       (effects (font (size 1.27 1.27)) hide)
     )
+    (property "Mfg" "KEMET" (id 4) (at 96.52 60.96 0)
+      (effects (font (size 1.27 1.27)) hide)
+    )
+    (property "PN" "C0402C104K8PAC7411" (id 5) (at 96.52 60.96 0)
+      (effects (font (size 1.27 1.27)) hide)
+    )
   )
   (symbol (lib_id "Device:C") (at 105.41 60.96 0) (mirror y) (unit 1)
@@
       (effects (font (size 1.27 1.27)) hide)
     )
+    (property "Mfg" "KEMET" (id 4) (at 105.41 60.96 0)
+      (effects (font (size 1.27 1.27)) hide)
+    )
+    (property "PN" "C0402C104K8PAC7411" (id 5) (at 105.41 60.96 0)
+      (effects (font (size 1.27 1.27)) hide)
+    )
   )
   (symbol (lib_id "Device:C") (at 251.46 72.39 0) (mirror y) (unit 1)
@@
     )
     (property "Datasheet" "~" (id 3) (at 251.46 72.39 0)
+      (effects (font (size 1.27 1.27)) hide)
+    )
+    (property "Mfg" "KEMET" (id 4) (at 251.46 72.39 0)
+      (effects (font (size 1.27 1.27)) hide)
+    )
+    (property "PN" "C0402C104K8PAC7411" (id 5) (at 251.46 72.39 0)
       (effects (font (size 1.27 1.27)) hide)
     )
@@
       (effects (font (size 1.27 1.27)) hide)
     )
-    (property "Mfg" "ISSI, Integrated Silicon Solution Inc" (id 6) (at -114.3 173.99 0)
+    (property "Mfg" "" (id 6) (at -114.3 173.99 0)
       (effects (font (size 1.27 1.27)) hide)
     )
@@
       (effects (font (size 1.524 1.524)) (justify right) hide)
     )
+    (property "PN" "LFE5U-12F-8BG256C" (id 4) (at 198.12 72.39 0)
+      (effects (font (size 1.27 1.27)) hide)
+    )
   )
