File: syzygy-flir-boson/kicad-src/syzygy-flir-boson.kicad_pcb (KiCad board)
At the start: 4 copper layers, 45 x 78 mm, 47 parts, among them J1 SYZYGY-STD, J2 Boson, J3 TagConnect, U1 TPS2061, U2 ATtiny44A-MMH, U3 INA219AxDCN

Commit message: syzygy-boson: Add BOM values to project
Parts:
- R15: value 10K -> 10k
Connections:
- J1 pad 37: Net-(J1-Pad37) -> unconnected-(J1-Pad37)
- J1 pad 38: Net-(J1-Pad38) -> unconnected-(J1-Pad38)
- U2 pad 10: no_connect_86 -> unconnected-(U2-Pad10)
- U2 pad 11: Net-(U2-Pad11) -> unconnected-(U2-Pad11)
- U2 pad 12: Net-(U2-Pad12) -> unconnected-(U2-Pad12)
- U2 pad 14: Net-(U2-Pad14) -> unconnected-(U2-Pad14)
- U2 pad 15: Net-(U2-Pad15) -> unconnected-(U2-Pad15)
- U2 pad 17: no_connect_87 -> unconnected-(U2-Pad17)
- U2 pad 18: no_connect_88 -> unconnected-(U2-Pad18)
- U2 pad 19: no_connect_89 -> unconnected-(U2-Pad19)
- U2 pad 2: Net-(U2-Pad2) -> unconnected-(U2-Pad2)
- U2 pad 3: Net-(U2-Pad3) -> unconnected-(U2-Pad3)
- U2 pad 4: Net-(U2-Pad4) -> unconnected-(U2-Pad4)
- U2 pad 6: no_connect_90 -> unconnected-(U2-Pad6)
- U2 pad 7: no_connect_91 -> unconnected-(U2-Pad7)
