File: syzygy-flir-boson/kicad-src/syzygy-flir-boson.kicad_sch (KiCad schematic)
At the start: 34 parts, among them J1 SYZYGY-STD, J2 Boson, U1 TPS2061, U3 INA219AxDCN

Commit message: syzygy-boson: Add BOM values to project
Parts:
- C1, C11, C13, C2, C5, C8: Mfg Samsung Electro-Mechanics -> Yageo; PN CL05F104ZO5NNNC -> CC0402JRX7R7BB104
- C4, C7: Mfg (none) -> Lelon; PN (none) -> VZS151M1ATR-0606
- H1, H2, H3, H4: Mfg (none) -> DNP
- J1: PN QTE-020-01-F-D-A -> QTE-020-01-F-D-A-K
- L1: Mfg (none) -> GLE; PN (none) -> GCNR5020-220MC
- R1, R10, R11, R2: PN RC0402JR-0710RL -> RC0402JR-0710KL
- R12, R8, R9: PN RC0402JR-0710RL -> RC0402JR-070RL
